File: KiCad LED Rings/Kicad LED Rings-V2/Kicad LED Rings_Circular_final_V2.kicad_pcb (KiCad board)
At the start: 4 copper layers, 30 x 30 mm, 27 parts, among them J1 Conn_01x02_Female, J2 Conn_01x02_Male, U1 LM3509SD_NOPB

Commit message: LED Ring PCB
Roated the MiniCAM LED Ring by 90 degrees.
Parts:
- added G***: LOGO, .Logo:Minicam_LED_Ring, B.Cu at (101.0, 80.3)
