File: KiCad LED Rings/Kicad LED Rings-V2/Kicad LED Rings.sch (KiCad schematic (older format))
At the start: 27 parts, among them J1 Conn_01x02_Female, J2 Conn_01x02_Male, U1 LM3509SD_NOPB

Commit message: Updated LED ring PCB
added part NO. of LM3509SD_NOPB
Parts:
- U1: PartNo. (none) -> LM3509SD_NOPB
Changed lines of the file:
@@
 F 2 "footprints:LM3509SD&slash_NOPB" H 3730 2290 60  0001 C CNN
 F 3 "" H 2030 2050 60  0000 C CNN
+F 4 "LM3509SD_NOPB" H 2030 2050 50  0001 C CNN "PartNo."
 	1    2030 2050
 	1    0    0    -1

Commit message: Updated LED Ring PCB
Changed '10uF 0603 25V' to '10uF 1210 50V'
Parts:
- C2: footprint .Capacitor_SMD:C_0603_1608Metric -> Capacitor:C_1210_3225Metric_L; PartNo. GRM188R61E106MA73J -> C1210C106K5RACTU
- R1, R4: value 10K -> 3K; PartNo. ERA-2AED103X -> ERA-2AEB302X
- R2: value 10K -> 9.5k; PartNo. ERA-2AED103X -> ERA-2AEB9531X
Changed lines of the file:
@@
 F 0 "C2" V 6191 2450 50  0000 C CNN
 F 1 "10uF" V 6282 2450 50  0000 C CNN
-F 2 ".Capacitor_SMD:C_0603_1608Metric" H 6458 2300 50  0001 C CNN
-F 3 "~" H 6420 2450 50  0001 C CNN
-F 4 "GRM188R61E106MA73J" V 6420 2450 50  0001 C CNN "PartNo."
+F 2 "Capacitor:C_1210_3225Metric_L" H 6458 2300 50  0001 C CNN
+F 3 "https://www.digikey.in/product-detail/en/kemet/C1210C106K5RACTU/399-11629-2-ND/4918882" H 6420 2450 50  0001 C CNN
+F 4 "C1210C106K5RACTU" V 6420 2450 50  0001 C CNN "PartNo."
 	1    6420 2450
 	0    1    1    0
@@
 P 1490 2610
 F 0 "R2" H 1558 2656 50  0000 L CNN
-F 1 "10K" H 1558 2565 50  0000 L CNN
+F 1 "9.5k" H 1558 2565 50  0000 L CNN
 F 2 "Resistor_SMD:R_0402_1005Metric" H 1490 2610 50  0001 C CNN
-F 3 "https://www.digikey.com/product-detail/en/panasonic-electronic-components/ERA-2AED103X/P10KDETR-ND/1706126" H 1490 2610 50  0001 C CNN
-F 4 "ERA-2AED103X" H 1550 2520 50  0001 C CNN "PartNo."
+F 3 "https://www.digikey.com/product-detail/en/panasonic-electronic-components/ERA-2AEB123X/P12KDCCT-ND/1706209" H 1490 2610 50  0001 C CNN
+F 4 "ERA-2AEB9531X" H 1550 2520 50  0001 C CNN "PartNo."
 	1    1490 2610
 	1    0    0    -1
@@
 F 2 "Resistor_SMD:R_0402_1005Metric" H 1820 2250 50  0001 C CNN
 F 3 "https://www.digikey.com/product-detail/en/panasonic-electronic-components/ERA-2AEB123X/P12KDCCT-ND/1706209" H 1820 2250 50  0001 C CNN
-F 4 "ERA-2AEB9531X" V 1770 2270 50  0000 C CNN "PartNo."
+F 4 "ERA-2AEB9531X" V 1770 2270 50  0001 C CNN "PartNo."
 	1    1820 2250
 	0    -1   -1   0
@@
 P 6680 4090
 F 0 "R1" H 6900 4100 50  0000 L CNN
-F 1 "10K" H 6740 4170 50  0000 L CNN
+F 1 "3K" H 6740 4170 50  0000 L CNN
 F 2 "Resistor_SMD:R_0402_1005Metric" H 6680 4090 50  0001 C CNN
-F 3 "https://www.digikey.com/product-detail/en/panasonic-electronic-components/ERA-2AED103X/P10KDETR-ND/1706126" H 6680 4090 50  0001 C CNN
-F 4 "ERA-2AED103X" H 6680 4090 50  0001 C CNN "PartNo."
+F 3 "https://www.digikey.in/product-detail/en/panasonic-electronic-components/ERA-2AEB302X/P3-0KDCTR-ND/1706016" H 6680 4090 50  0001 C CNN
+F 4 "ERA-2AEB302X" H 6680 4090 50  0001 C CNN "PartNo."
 	1    6680 4090
 	-1   0    0    1
@@
 P 7040 4090
 F 0 "R4" H 6840 4070 50  0000 L CNN
-F 1 "10K" H 6830 4160 50  0000 L CNN
+F 1 "3K" H 6830 4160 50  0000 L CNN
 F 2 "Resistor_SMD:R_0402_1005Metric" H 7040 4090 50  0001 C CNN
-F 3 "https://www.digikey.com/product-detail/en/panasonic-electronic-components/ERA-2AED103X/P10KDETR-ND/1706126" H 7040 4090 50  0001 C CNN
-F 4 "ERA-2AED103X" H 7040 4090 50  0001 C CNN "PartNo."
+F 3 "https://www.digikey.in/product-detail/en/panasonic-electronic-components/ERA-2AEB302X/P3-0KDCTR-ND/1706016" H 7040 4090 50  0001 C CNN
+F 4 "ERA-2AEB302X" H 7040 4090 50  0001 C CNN "PartNo."
 	1    7040 4090
 	-1   0    0    1

Commit message: Upldated LED ring PCB
Changed 10uF Cout to C2012X5R1E225M125AC;
Changed 10uH inductor to NRS4012T100MDGJ;
Parts:
- C2: value 10uF -> 2.2uF; footprint Capacitor:C_1210_3225Metric_L -> .Capacitor:C_0805_2012Metric_L; PartNo. C1210C106K5RACTU -> C2012X5R1E225M125AC
- L1: footprint footprints:VLF4012AT-100MR79 -> footprints:NRS4012T100MDGJ; symbol Kicad-LED-Rings-rescue:ADL3225V-470MT-TL000-.Inductor-Kicad-LED-Rings-rescue -> 2020-07-30_23-38-29:NRS4012T100MDGJ; PartNo. VLF4012AT-100MR79 -> NRS4012T100MDGJ
Connections:
- wire segments 53 -> 52
Changed lines of the file:
@@
 P 6420 2450
 F 0 "C2" V 6191 2450 50  0000 C CNN
-F 1 "10uF" V 6282 2450 50  0000 C CNN
-F 2 "Capacitor:C_1210_3225Metric_L" H 6458 2300 50  0001 C CNN
-F 3 "https://www.digikey.in/product-detail/en/kemet/C1210C106K5RACTU/399-11629-2-ND/4918882" H 6420 2450 50  0001 C CNN
-F 4 "C1210C106K5RACTU" V 6420 2450 50  0001 C CNN "PartNo."
+F 1 "2.2uF" V 6282 2450 50  0000 C CNN
+F 2 ".Capacitor:C_0805_2012Metric_L" H 6458 2300 50  0001 C CNN
+F 3 "https://www.digikey.com/product-detail/en/tdk-corporation/C2012X5R1E225M125AC/445-7630-2-ND/2733065" H 6420 2450 50  0001 C CNN
+F 4 "C2012X5R1E225M125AC" V 6420 2450 50  0001 C CNN "PartNo."
 	1    6420 2450
 	0    1    1    0
@@
 $EndComp
 $Comp
-L Kicad-LED-Rings-rescue:ADL3225V-470MT-TL000-.Inductor-Kicad-LED-Rings-rescue L1
+L 2020-07-30_23-38-29:NRS4012T100MDGJ L1
 U 1 1 5E8B36F1
-P 5700 2550
-F 0 "L1" V 5560 2540 50  0000 C CNN
-F 1 "10uH" V 5650 2450 50  0000 L CNN
-F 2 "footprints:VLF4012AT-100MR79" H 5630 2490 50  0001 C CNN
-F 3 "https://product.tdk.com/info/en/catalog/datasheets/inductor_automotive_decoupling_adl3225v_en.pdf" H 5700 2550 50  0001 C CNN
-F 4 "VLF4012AT-100MR79" V 5640 2550 50  0001 C CNN "PartNo."
-	1    5700 2550
-	0    -1   -1   0
+P 5450 2650
+F 0 "L1" H 5650 2600 50  0000 C CNN
+F 1 "10uH" H 5700 2600 50  0000 L CNN
+F 2 "footprints:NRS4012T100MDGJ" H 5380 2590 50  0001 C CNN
+F 3 "https://www.digikey.com/product-detail/en/taiyo-yuden/NRS4012T100MDGJ/587-2878-1-ND/2648998" H 5450 2650 50  0001 C CNN
+F 4 "NRS4012T100MDGJ" V 5390 2650 50  0001 C CNN "PartNo."
+	1    5450 2650
+	1    0    0    -1
 $EndComp
 $Comp
@@
 L Kicad-LED-Rings-rescue:+5V-power #PWR04
 U 1 1 5E8B7DFD
-P 5970 2550
-F 0 "#PWR04" H 5970 2400 50  0001 C CNN
-F 1 "+5V" V 5985 2678 50  0000 L CNN
-F 2 "" H 5970 2550 50  0001 C CNN
-F 3 "" H 5970 2550 50  0001 C CNN
-	1    5970 2550
+P 6050 2650
+F 0 "#PWR04" H 6050 2500 50  0001 C CNN
+F 1 "+5V" V 6100 2550 50  0000 L CNN
+F 2 "" H 6050 2650 50  0001 C CNN
+F 3 "" H 6050 2650 50  0001 C CNN
+	1    6050 2650
 	0    1    1    0
 $EndComp
-Wire Wire Line
-	5800 2550 5970 2550
 Wire Wire Line
 	5430 2450 6320 2450
@@
 $EndComp
 Wire Wire Line
-	5450 3070 5450 2550
-Connection ~ 5450 2550
-Wire Wire Line
-	5450 2550 5600 2550
+	5450 3070 5450 2650
 Text GLabel 6130 3070 2    50   Input ~ 0
 OVP
@@
 Wire Wire Line
 	4650 1390 4720 1390
+Connection ~ 5450 2650
+Wire Wire Line
+	5450 2650 5450 2550
 $EndSCHEMATC

Commit message: Modified PCB layout
Parts:
- L1: symbol 2020-07-30_23-38-29:NRS4012T100MDGJ -> Kicad-LED-Rings-rescue:NRS4012T100MDGJ-2020-07-30_23-38-29
- renumbered D8 to D11, D15 to D12, D6 to D13, D4 to D14, D13 to D15, D2 to D16, D11 to D17, D12 to D2, D5 to D4, D14 to D5, D7 to D6, D9 to D7, D16 to D8, D17 to D9
Connections:
- net at U1.1 (MAIN): now also D1.1 (K); no longer D16.1 (K)
- net at U1.2 (SUB/FB): now also D16.1 (K); no longer D1.1 (K)
Changed lines of the file:
@@
 EESchema Schematic File Version 4
-LIBS:Kicad LED Rings-cache
 EELAYER 30 0
 EELAYER END
@@
 encoding utf-8
 Sheet 1 1
-Title ""
-Date ""
-Rev ""
-Comp ""
+Title "MiniCAM LED Ring"
+Date "2020-07-31"
+Rev "v0.2"
+Comp "Aharoni Lab"
 Comment1 ""
 Comment2 ""
@@
 Comment4 ""
 $EndDescr
-$Comp
-L Kicad-LED-Rings-rescue:LM3509SD_NOPB-2020-04-05_20-57-04 U1
-U 1 1 5E8A688C
-P 2030 2050
-F 0 "U1" H 3730 2437 60  0000 C CNN
-F 1 "LM3509SD_NOPB" H 3730 2331 60  0000 C CNN
-F 2 "footprints:LM3509SD&slash_NOPB" H 3730 2290 60  0001 C CNN
-F 3 "" H 2030 2050 60  0000 C CNN
-F 4 "LM3509SD_NOPB" H 2030 2050 50  0001 C CNN "PartNo."
-	1    2030 2050
-	1    0    0    -1
-$EndComp
 $Comp
 L Kicad-LED-Rings-rescue:+5V-power #PWR03
@@
 $EndComp
 $Comp
-L 2020-07-30_23-38-29:NRS4012T100MDGJ L1
+L Kicad-LED-Rings-rescue:NRS4012T100MDGJ-2020-07-30_23-38-29 L1
 U 1 1 5E8B36F1
 P 5450 2650
@@
 	6680 4190 6680 4380
 $Comp
-L Kicad-LED-Rings-rescue:BAT760,115-BAT760_115 D11
+L Kicad-LED-Rings-rescue:BAT760,115-BAT760_115 D17
 U 1 1 5E8AEDAE
 P 5690 3070
-F 0 "D11" H 5690 3287 50  0000 C CNN
+F 0 "D17" H 5690 3287 50  0000 C CNN
 F 1 "D_Schottky" H 5690 3196 50  0000 C CNN
 F 2 "BAT760_115:SOD323(F)" H 5690 3070 50  0001 C CNN
@@
 OVP
 $Comp
-L Kicad-LED-Rings-rescue:LED_Small_ALT-Device D2
+L Kicad-LED-Rings-rescue:LED_Small_ALT-Device D16
 U 1 1 5E8B124A
 P 2790 1390
-F 0 "D2" H 2790 1625 50  0000 C CNN
+F 0 "D16" H 2790 1625 50  0000 C CNN
 F 1 "LED_Small_ALT" H 2790 1534 50  0000 C CNN
 F 2 "LED_SMD:LED_0603_1608Metric" V 2790 1390 50  0001 C CNN
@@
 $EndComp
 $Comp
-L Kicad-LED-Rings-rescue:LED_Small_ALT-Device D4
+L Kicad-LED-Rings-rescue:LED_Small_ALT-Device D14
 U 1 1 5E8B1A2E
 P 3280 1390
-F 0 "D4" H 3280 1625 50  0000 C CNN
+F 0 "D14" H 3280 1625 50  0000 C CNN
 F 1 "LED_Small_ALT" H 3280 1534 50  0000 C CNN
 F 2 "LED_SMD:LED_0603_1608Metric" V 3280 1390 50  0001 C CNN
@@
 $EndComp
 $Comp
-L Kicad-LED-Rings-rescue:LED_Small_ALT-Device D6
+L Kicad-LED-Rings-rescue:LED_Small_ALT-Device D13
 U 1 1 5E8B2164
 P 3550 1390
-F 0 "D6" H 3550 1625 50  0000 C CNN
+F 0 "D13" H 3550 1625 50  0000 C CNN
 F 1 "LED_Small_ALT" H 3550 1534 50  0000 C CNN
 F 2 "LED_SMD:LED_0603_1608Metric" V 3550 1390 50  0001 C CNN
@@
 $EndComp
 $Comp
-L Kicad-LED-Rings-rescue:LED_Small_ALT-Device D8
+L Kicad-LED-Rings-rescue:LED_Small_ALT-Device D11
 U 1 1 5E8B273B
 P 4040 1390
-F 0 "D8" H 4040 1625 50  0000 C CNN
+F 0 "D11" H 4040 1625 50  0000 C CNN
 F 1 "LED_Small_ALT" H 4040 1534 50  0000 C CNN
 F 2 "LED_SMD:LED_0603_1608Metric" V 4040 1390 50  0001 C CNN
@@
 $EndComp
 $Comp
-L Kicad-LED-Rings-rescue:LED_Small_ALT-Device D9
+L Kicad-LED-Rings-rescue:LED_Small_ALT-Device D7
 U 1 1 5E8B5CB2
 P 4290 920
-F 0 "D9" H 4290 1155 50  0000 C CNN
+F 0 "D7" H 4290 1155 50  0000 C CNN
 F 1 "LED_Small_ALT" H 4290 1064 50  0000 C CNN
 F 2 "LED_SMD:LED_0603_1608Metric" V 4290 920 50  0001 C CNN
@@
 $EndComp
 $Comp
-L Kicad-LED-Rings-rescue:LED_Small_ALT-Device D7
+L Kicad-LED-Rings-rescue:LED_Small_ALT-Device D6
 U 1 1 5E8B5CA8
 P 4050 920
-F 0 "D7" H 4050 1155 50  0000 C CNN
+F 0 "D6" H 4050 1155 50  0000 C CNN
 F 1 "LED_Small_ALT" H 4050 1064 50  0000 C CNN
 F 2 "LED_SMD:LED_0603_1608Metric" V 4050 920 50  0001 C CNN
@@
 $EndComp
 $Comp
-L Kicad-LED-Rings-rescue:LED_Small_ALT-Device D5
+L Kicad-LED-Rings-rescue:LED_Small_ALT-Device D4
 U 1 1 5E8B5C9E
 P 3550 920
-F 0 "D5" H 3550 1155 50  0000 C CNN
+F 0 "D4" H 3550 1155 50  0000 C CNN
 F 1 "LED_Small_ALT" H 3550 1064 50  0000 C CNN
 F 2 "LED_SMD:LED_0603_1608Metric" V 3550 920 50  0001 C CNN
@@
 Wire Wire Line
 	2030 2150 1930 2150
-Wire Wire Line
-	1930 2150 1930 920
-Wire Wire Line
-	1930 920  2690 920
-Wire Wire Line
-	2690 1390 2030 1390
-Wire Wire Line
-	2030 1390 2030 2050
 Text GLabel 5430 2150 2    50   Input ~ 0
 SCL
@@
 	6870 3820 7040 3820
 $Comp
-L Kicad-LED-Rings-rescue:LED_Small_ALT-Device D12
+L Kicad-LED-Rings-rescue:LED_Small_ALT-Device D2
 U 1 1 5F10EE3C
 P 3030 920
-F 0 "D12" H 3030 1155 50  0000 C CNN
+F 0 "D2" H 3030 1155 50  0000 C CNN
 F 1 "LED_Small_ALT" H 3030 1064 50  0000 C CNN
 F 2 "LED_SMD:LED_0603_1608Metric" V 3030 920 50  0001 C CNN
@@
 $EndComp
 $Comp
-L Kicad-LED-Rings-rescue:LED_Small_ALT-Device D14
+L Kicad-LED-Rings-rescue:LED_Small_ALT-Device D5
 U 1 1 5F10F69F
 P 3790 920
-F 0 "D14" H 3790 1155 50  0000 C CNN
+F 0 "D5" H 3790 1155 50  0000 C CNN
 F 1 "LED_Small_ALT" H 3790 1064 50  0000 C CNN
 F 2 "LED_SMD:LED_0603_1608Metric" V 3790 920 50  0001 C CNN
@@
 $EndComp
 $Comp
-L Kicad-LED-Rings-rescue:LED_Small_ALT-Device D16
+L Kicad-LED-Rings-rescue:LED_Small_ALT-Device D8
 U 1 1 5F110CD4
 P 4540 920
-F 0 "D16" H 4540 1155 50  0000 C CNN
+F 0 "D8" H 4540 1155 50  0000 C CNN
 F 1 "LED_Small_ALT" H 4540 1064 50  0000 C CNN
 F 2 "LED_SMD:LED_0603_1608Metric" V 4540 920 50  0001 C CNN
@@
 $EndComp
 $Comp
-L Kicad-LED-Rings-rescue:LED_Small_ALT-Device D13
+L Kicad-LED-Rings-rescue:LED_Small_ALT-Device D15
 U 1 1 5F1112DB
 P 3030 1390
-F 0 "D13" H 3030 1625 50  0000 C CNN
+F 0 "D15" H 3030 1625 50  0000 C CNN
 F 1 "LED_Small_ALT" H 3030 1534 50  0000 C CNN
 F 2 "LED_SMD:LED_0603_1608Metric" V 3030 1390 50  0001 C CNN
@@
 $EndComp
 $Comp
-L Kicad-LED-Rings-rescue:LED_Small_ALT-Device D15
+L Kicad-LED-Rings-rescue:LED_Small_ALT-Device D12
 U 1 1 5F1120C3
 P 3790 1390
-F 0 "D15" H 3790 1625 50  0000 C CNN
+F 0 "D12" H 3790 1625 50  0000 C CNN
 F 1 "LED_Small_ALT" H 3790 1534 50  0000 C CNN
 F 2 "LED_SMD:LED_0603_1608Metric" V 3790 1390 50  0001 C CNN
@@
 $EndComp
 $Comp
-L Kicad-LED-Rings-rescue:LED_Small_ALT-Device D17
+L Kicad-LED-Rings-rescue:LED_Small_ALT-Device D9
 U 1 1 5F11304A
 P 4550 1390
-F 0 "D17" H 4550 1625 50  0000 C CNN
+F 0 "D9" H 4550 1625 50  0000 C CNN
 F 1 "LED_Small_ALT" H 4550 1534 50  0000 C CNN
 F 2 "LED_SMD:LED_0603_1608Metric" V 4550 1390 50  0001 C CNN
@@
 Wire Wire Line
 	5450 2650 5450 2550
+$Comp
+L Kicad-LED-Rings-rescue:LM3509SD_NOPB-2020-04-05_20-57-04 U1
+U 1 1 5E8A688C
+P 2030 2050
+F 0 "U1" H 3730 2437 60  0000 C CNN
+F 1 "LM3509SD_NOPB" H 3730 2331 60  0000 C CNN
+F 2 "footprints:LM3509SD&slash_NOPB" H 3730 2290 60  0001 C CNN
+F 3 "" H 2030 2050 60  0000 C CNN
+F 4 "LM3509SD_NOPB" H 2030 2050 50  0001 C CNN "PartNo."
+	1    2030 2050
+	1    0    0    -1
+$EndComp
+Wire Wire Line
+	1930 1390 1930 2150
+Wire Wire Line
+	1930 1390 2690 1390
+Wire Wire Line
+	2030 2050 2030 920
+Wire Wire Line
+	2030 920  2690 920
 $EndSCHEMATC
