File: KiCad LED Rings/Kicad LED Rings-V2/_autosave-Kicad LED Rings.sch (KiCad schematic (older format))
At the start: 27 parts, among them J1 Conn_01x02_Female, J2 Conn_01x02_Male, U1 LM3509SD_NOPB

Commit message: Upldated MiniCAM
Removed the short footprint of  10uH inductor NRS4012T100MDGJ;
Corrected the wroing footprint of 10uH inductor and saved the corrected footprint as 'NRS4012T100MDGJ_Corrected_09012020' in C:\Users\Changliang Guo\Desktop\GitHub\MiniCAM\KiCad LED Rings\10uH Inductor
Parts:
- C1, C2: symbol Kicad-LED-Rings-rescue:GRM033R60J105MEA2D-.Capacitor-Kicad-LED-Rings-rescue -> Kicad-LED-Rings-rescue:GRM033R60J105MEA2D-.Capacitor-Kicad-LED-Rings-rescue-Kicad-LED-Rings-rescue
- D1, D10, D11, D12, D13, D14, D15, D16, D2, D3, D4, D5, D6, D7, D8, D9: symbol Kicad-LED-Rings-rescue:LED_Small_ALT-Device -> Kicad-LED-Rings-rescue:LED_Small_ALT-Device-Kicad-LED-Rings-rescue
- D17: symbol Kicad-LED-Rings-rescue:BAT760,115-BAT760_115 -> Kicad-LED-Rings-rescue:BAT760,115-BAT760_115-Kicad-LED-Rings-rescue
- J1: symbol Kicad-LED-Rings-rescue:Conn_01x03_Female-Connector -> Kicad-LED-Rings-rescue:Conn_01x03_Female-Connector-Kicad-LED-Rings-rescue
- J2: symbol Kicad-LED-Rings-rescue:Conn_01x02_Male-Connector -> Kicad-LED-Rings-rescue:Conn_01x02_Male-Connector-Kicad-LED-Rings-rescue
- R1, R2, R3, R4: symbol Kicad-LED-Rings-rescue:R_Small-Device -> Kicad-LED-Rings-rescue:R_Small-Device-Kicad-LED-Rings-rescue
- U1: symbol Kicad-LED-Rings-rescue:LM3509SD_NOPB-2020-04-05_20-57-04 -> Kicad-LED-Rings-rescue:LM3509SD_NOPB-2020-04-05_20-57-04-Kicad-LED-Rings-rescue
Changed lines of the file:
@@
 encoding utf-8
 Sheet 1 1
-Title ""
-Date ""
-Rev ""
-Comp ""
+Title "MiniCAM LED Ring"
+Date "2020-07-31"
+Rev "v0.2"
+Comp "Aharoni Lab"
 Comment1 ""
 Comment2 ""
@@
 $EndDescr
 $Comp
-L Kicad-LED-Rings-rescue:+5V-power #PWR03
+L Kicad-LED-Rings-rescue:+5V-power-Kicad-LED-Rings-rescue #PWR03
 U 1 1 5E8AAF06
 P 5970 2350
@@
 $EndComp
 $Comp
-L Kicad-LED-Rings-rescue:GRM033R60J105MEA2D-.Capacitor-Kicad-LED-Rings-rescue C2
+L Kicad-LED-Rings-rescue:GRM033R60J105MEA2D-.Capacitor-Kicad-LED-Rings-rescue-Kicad-LED-Rings-rescue C2
 U 1 1 5E8B056A
 P 6420 2450
@@
 $EndComp
 $Comp
-L Kicad-LED-Rings-rescue:R_Small-Device R2
+L Kicad-LED-Rings-rescue:R_Small-Device-Kicad-LED-Rings-rescue R2
 U 1 1 5E8B1987
 P 1490 2610
@@
 $EndComp
 $Comp
-L Kicad-LED-Rings-rescue:R_Small-Device R3
+L Kicad-LED-Rings-rescue:R_Small-Device-Kicad-LED-Rings-rescue R3
 U 1 1 5E8B1D0A
 P 1820 2250
@@
 $EndComp
 $Comp
-L Kicad-LED-Rings-rescue:R_Small-Device R1
+L Kicad-LED-Rings-rescue:R_Small-Device-Kicad-LED-Rings-rescue R1
 U 1 1 5E8B20E8
 P 6680 4090
@@
 $EndComp
 $Comp
-L Kicad-LED-Rings-rescue:GRM033R60J105MEA2D-.Capacitor-Kicad-LED-Rings-rescue C1
+L Kicad-LED-Rings-rescue:GRM033R60J105MEA2D-.Capacitor-Kicad-LED-Rings-rescue-Kicad-LED-Rings-rescue C1
 U 1 1 5E8B4731
 P 5860 2170
@@
 	5430 2550 5450 2550
 $Comp
-L Kicad-LED-Rings-rescue:+5V-power #PWR04
+L Kicad-LED-Rings-rescue:+5V-power-Kicad-LED-Rings-rescue #PWR04
 U 1 1 5E8B7DFD
 P 6050 2650
@@
 	5430 2450 6320 2450
 $Comp
-L Kicad-LED-Rings-rescue:GND-power #PWR06
+L Kicad-LED-Rings-rescue:GND-power-Kicad-LED-Rings-rescue #PWR06
 U 1 1 5E8B9C78
 P 6670 2600
@@
 	5860 2350 5970 2350
 $Comp
-L Kicad-LED-Rings-rescue:GND-power #PWR05
+L Kicad-LED-Rings-rescue:GND-power-Kicad-LED-Rings-rescue #PWR05
 U 1 1 5E8BCC8C
 P 6230 2070
@@
 	5860 2070 6230 2070
 $Comp
-L Kicad-LED-Rings-rescue:GND-power #PWR02
+L Kicad-LED-Rings-rescue:GND-power-Kicad-LED-Rings-rescue #PWR02
 U 1 1 5E8BDC5C
 P 5430 1910
@@
 	2030 2250 1920 2250
 $Comp
-L Kicad-LED-Rings-rescue:GND-power #PWR01
+L Kicad-LED-Rings-rescue:GND-power-Kicad-LED-Rings-rescue #PWR01
 U 1 1 5E8A8FD0
 P 1470 2250
@@
 	6680 4190 6680 4380
 $Comp
-L Kicad-LED-Rings-rescue:BAT760,115-BAT760_115 D17
+L Kicad-LED-Rings-rescue:BAT760,115-BAT760_115-Kicad-LED-Rings-rescue D17
 U 1 1 5E8AEDAE
 P 5690 3070
@@
 OVP
 $Comp
-L Kicad-LED-Rings-rescue:LED_Small_ALT-Device D16
+L Kicad-LED-Rings-rescue:LED_Small_ALT-Device-Kicad-LED-Rings-rescue D16
 U 1 1 5E8B124A
 P 2790 1390
@@
 $EndComp
 $Comp
-L Kicad-LED-Rings-rescue:LED_Small_ALT-Device D14
+L Kicad-LED-Rings-rescue:LED_Small_ALT-Device-Kicad-LED-Rings-rescue D14
 U 1 1 5E8B1A2E
 P 3280 1390
@@
 $EndComp
 $Comp
-L Kicad-LED-Rings-rescue:LED_Small_ALT-Device D13
+L Kicad-LED-Rings-rescue:LED_Small_ALT-Device-Kicad-LED-Rings-rescue D13
 U 1 1 5E8B2164
 P 3550 1390
@@
 $EndComp
 $Comp
-L Kicad-LED-Rings-rescue:LED_Small_ALT-Device D11
+L Kicad-LED-Rings-rescue:LED_Small_ALT-Device-Kicad-LED-Rings-rescue D11
 U 1 1 5E8B273B
 P 4040 1390
@@
 $EndComp
 $Comp
-L Kicad-LED-Rings-rescue:LED_Small_ALT-Device D10
+L Kicad-LED-Rings-rescue:LED_Small_ALT-Device-Kicad-LED-Rings-rescue D10
 U 1 1 5E8B2DC2
 P 4310 1390
@@
 $EndComp
 $Comp
-L Kicad-LED-Rings-rescue:LED_Small_ALT-Device D7
+L Kicad-LED-Rings-rescue:LED_Small_ALT-Device-Kicad-LED-Rings-rescue D7
 U 1 1 5E8B5CB2
 P 4290 920
@@
 $EndComp
 $Comp
-L Kicad-LED-Rings-rescue:LED_Small_ALT-Device D6
+L Kicad-LED-Rings-rescue:LED_Small_ALT-Device-Kicad-LED-Rings-rescue D6
 U 1 1 5E8B5CA8
 P 4050 920
@@
 $EndComp
 $Comp
-L Kicad-LED-Rings-rescue:LED_Small_ALT-Device D4
+L Kicad-LED-Rings-rescue:LED_Small_ALT-Device-Kicad-LED-Rings-rescue D4
 U 1 1 5E8B5C9E
 P 3550 920
@@
 $EndComp
 $Comp
-L Kicad-LED-Rings-rescue:LED_Small_ALT-Device D3
+L Kicad-LED-Rings-rescue:LED_Small_ALT-Device-Kicad-LED-Rings-rescue D3
 U 1 1 5E8B5C94
 P 3280 920
@@
 $EndComp
 $Comp
-L Kicad-LED-Rings-rescue:LED_Small_ALT-Device D1
+L Kicad-LED-Rings-rescue:LED_Small_ALT-Device-Kicad-LED-Rings-rescue D1
 U 1 1 5E8B5C8A
 P 2790 920
@@
 SDA
 $Comp
-L Kicad-LED-Rings-rescue:Conn_01x03_Female-Connector J1
+L Kicad-LED-Rings-rescue:Conn_01x03_Female-Connector-Kicad-LED-Rings-rescue J1
 U 1 1 5E8C7898
 P 3530 3720
@@
 $EndComp
 $Comp
-L Kicad-LED-Rings-rescue:Conn_01x02_Male-Connector J2
+L Kicad-LED-Rings-rescue:Conn_01x02_Male-Connector-Kicad-LED-Rings-rescue J2
 U 1 1 5E8C7DAA
 P 5200 3680
@@
 $EndComp
 $Comp
-L Kicad-LED-Rings-rescue:GND-power #PWR0101
+L Kicad-LED-Rings-rescue:GND-power-Kicad-LED-Rings-rescue #PWR0101
 U 1 1 5E8C8610
 P 3330 3620
@@
 $EndComp
 $Comp
-L Kicad-LED-Rings-rescue:+5V-power #PWR0102
+L Kicad-LED-Rings-rescue:+5V-power-Kicad-LED-Rings-rescue #PWR0102
 U 1 1 5E8C8FD0
 P 3210 3720
@@
 	5790 3070 6130 3070
 $Comp
-L Kicad-LED-Rings-rescue:+2V8-power #PWR011
+L Kicad-LED-Rings-rescue:+2V8-power-Kicad-LED-Rings-rescue #PWR011
 U 1 1 5E9546A9
 P 1320 2350
@@
 $EndComp
 $Comp
-L Kicad-LED-Rings-rescue:R_Small-Device R4
+L Kicad-LED-Rings-rescue:R_Small-Device-Kicad-LED-Rings-rescue R4
 U 1 1 5E95957D
 P 7040 4090
@@
 	7040 3820 7040 3990
 $Comp
-L Kicad-LED-Rings-rescue:+2V8-power #PWR012
+L Kicad-LED-Rings-rescue:+2V8-power-Kicad-LED-Rings-rescue #PWR012
 U 1 1 5E95FB55
 P 6870 3820
@@
 $EndComp
 $Comp
-L Kicad-LED-Rings-rescue:+2V8-power #PWR0103
+L Kicad-LED-Rings-rescue:+2V8-power-Kicad-LED-Rings-rescue #PWR0103
 U 1 1 5EA52B66
 P 3210 3820
@@
 	6870 3820 7040 3820
 $Comp
-L Kicad-LED-Rings-rescue:LED_Small_ALT-Device D2
+L Kicad-LED-Rings-rescue:LED_Small_ALT-Device-Kicad-LED-Rings-rescue D2
 U 1 1 5F10EE3C
 P 3030 920
@@
 $EndComp
 $Comp
-L Kicad-LED-Rings-rescue:LED_Small_ALT-Device D5
+L Kicad-LED-Rings-rescue:LED_Small_ALT-Device-Kicad-LED-Rings-rescue D5
 U 1 1 5F10F69F
 P 3790 920
@@
 $EndComp
 $Comp
-L Kicad-LED-Rings-rescue:LED_Small_ALT-Device D8
+L Kicad-LED-Rings-rescue:LED_Small_ALT-Device-Kicad-LED-Rings-rescue D8
 U 1 1 5F110CD4
 P 4540 920
@@
 $EndComp
 $Comp
-L Kicad-LED-Rings-rescue:LED_Small_ALT-Device D15
+L Kicad-LED-Rings-rescue:LED_Small_ALT-Device-Kicad-LED-Rings-rescue D15
 U 1 1 5F1112DB
 P 3030 1390
@@
 $EndComp
 $Comp
-L Kicad-LED-Rings-rescue:LED_Small_ALT-Device D12
+L Kicad-LED-Rings-rescue:LED_Small_ALT-Device-Kicad-LED-Rings-rescue D12
 U 1 1 5F1120C3
 P 3790 1390
@@
 $EndComp
 $Comp
-L Kicad-LED-Rings-rescue:LED_Small_ALT-Device D9
+L Kicad-LED-Rings-rescue:LED_Small_ALT-Device-Kicad-LED-Rings-rescue D9
 U 1 1 5F11304A
 P 4550 1390
@@
 	5450 2650 5450 2550
 $Comp
-L Kicad-LED-Rings-rescue:LM3509SD_NOPB-2020-04-05_20-57-04 U1
+L Kicad-LED-Rings-rescue:LM3509SD_NOPB-2020-04-05_20-57-04-Kicad-LED-Rings-rescue U1
 U 1 1 5E8A688C
 P 2030 2050

Commit message: Updated LED ring pcb
Corrected the messed up schematics and footprints
Regenerated the Gerber files, position files, and drill files
Parts:
- L1: symbol Kicad-LED-Rings-rescue:NRS4012T100MDGJ-2020-07-30_23-38-29 -> LED_Ring-rescue:NRS4012T100MDGJ-2020-07-30_23-38-29
Connections:
- net at D17.2 (A), U1.6 (SW): no longer L1.2
Changed lines of the file:
@@
 $EndComp
 $Comp
-L Kicad-LED-Rings-rescue:NRS4012T100MDGJ-2020-07-30_23-38-29 L1
+L LED_Ring-rescue:NRS4012T100MDGJ-2020-07-30_23-38-29 L1
 U 1 1 5E8B36F1
 P 5450 2650
@@
 	1    0    0    -1
 $EndComp
-Wire Wire Line
-	5450 3070 5450 2650
 Text GLabel 6130 3070 2    50   Input ~ 0
 OVP
@@
 Wire Wire Line
 	4650 1390 4720 1390
-Connection ~ 5450 2650
-Wire Wire Line
-	5450 2650 5450 2550
 $Comp
 L Kicad-LED-Rings-rescue:LM3509SD_NOPB-2020-04-05_20-57-04-Kicad-LED-Rings-rescue U1
@@
 Wire Wire Line
 	2030 920  2690 920
+Wire Wire Line
+	5450 2550 5450 3070
 $EndSCHEMATC
