File: KiCad LED Rings/Kicad LED Rings-V2/LED_Ring.sch (KiCad schematic (older format))
At the start: 27 parts, among them J1 Conn_01x02_Female, J2 Conn_01x02_Male, U1 LM3509SD_NOPB

Commit message: updated led ring pcb board
Parts:
- C1: footprint .Capacitor_SMD:C_0603_1608Metric -> .Capacitor:C_0603_1608Metric_L; symbol Kicad-LED-Rings-rescue:GRM033R60J105MEA2D-.Capacitor-Kicad-LED-Rings-rescue -> Kicad-LED-Rings-rescue:GRM033R60J105MEA2D-.Capacitor-Kicad-LED-Rings-rescue-Kicad-LED-Rings-rescue
- C2: symbol Kicad-LED-Rings-rescue:GRM033R60J105MEA2D-.Capacitor-Kicad-LED-Rings-rescue -> Kicad-LED-Rings-rescue:GRM033R60J105MEA2D-.Capacitor-Kicad-LED-Rings-rescue-Kicad-LED-Rings-rescue
- D1, D10, D11, D12, D13, D14, D15, D16, D2, D3, D4, D5, D6, D7, D8, D9: footprint LED_SMD:LED_0603_1608Metric -> .LED:LED_0603_1608Metric; symbol Kicad-LED-Rings-rescue:LED_Small_ALT-Device -> Kicad-LED-Rings-rescue:LED_Small_ALT-Device-Kicad-LED-Rings-rescue
- D17: symbol Kicad-LED-Rings-rescue:BAT760,115-BAT760_115 -> Kicad-LED-Rings-rescue:BAT760,115-BAT760_115-Kicad-LED-Rings-rescue
- J1: symbol Kicad-LED-Rings-rescue:Conn_01x03_Female-Connector -> Kicad-LED-Rings-rescue:Conn_01x03_Female-Connector-Kicad-LED-Rings-rescue
- J2: symbol Kicad-LED-Rings-rescue:Conn_01x02_Male-Connector -> Kicad-LED-Rings-rescue:Conn_01x02_Male-Connector-Kicad-LED-Rings-rescue
- L1: footprint footprints:NRS4012T100MDGJ -> .Inductor:NR3015T1R5N; symbol Kicad-LED-Rings-rescue:NRS4012T100MDGJ-2020-07-30_23-38-29 -> LED_Ring-rescue:NRS4012T100MDGJ-2020-07-30_23-38-29
- R1, R2, R3, R4: footprint Resistor_SMD:R_0402_1005Metric -> .Resistor:R_0402_1005Metric_ERJ_L; symbol Kicad-LED-Rings-rescue:R_Small-Device -> Kicad-LED-Rings-rescue:R_Small-Device-Kicad-LED-Rings-rescue
- U1: footprint footprints:LM3509SD&slash_NOPB -> .LM3509SDNOPB:LM3509SDNOPB; symbol Kicad-LED-Rings-rescue:LM3509SD_NOPB-2020-04-05_20-57-04 -> Kicad-LED-Rings-rescue:LM3509SD_NOPB-2020-04-05_20-57-04-Kicad-LED-Rings-rescue
Connections:
- net at D17.2 (A), U1.6 (SW): no longer L1.2
